File: smartportsd-smd.kicad_pcb (KiCad board)
At the start: 2 copper layers, 45.4 x 52.1 mm, 25 parts, among them J1 DB19_Plug, J2 ICSP, J3 SD_Card_Push_Pull, SW1 SW_SPST, U1 ATmega328P-A, U2 4050, U3 AMS1117-3.3, Y1 16MHz

Commit message: Version 1.1
Parts:
- J1: footprint Tersteeg:DSUB-19_Male_Vertical_P2.77x2.84mm_MountingHoles -> Tersteeg:DSUB-19_Male_Vertical_P2.77x2.84mm_Narrow_MountingHoles
- moved J2 17.8 mm to (170.6, 96.9)
- moved R2 12.8 mm to (172.8, 90.2), turned to 90 degrees
- moved SW1 7.45 mm to (168.8, 91.2)
- moved C1 3.84 mm to (171.7, 110.5), turned to -90 degrees
- moved R3 3.27 mm to (172.8, 85.8), turned to -90 degrees
- moved D1 2.67 mm to (168.8, 85.0)
- moved J1 2.24 mm to (167.2, 126.8)
- moved R4 1.81 mm to (165.5, 96.0)
- moved R5 1.81 mm to (165.5, 98.0)
- moved R8 1.81 mm to (165.5, 94.0)
- moved R6 1.37 mm to (165.5, 101.1)
- moved R7 1.37 mm to (165.5, 103.1)
- moved C5 0.81 mm to (167.6, 107.4)
- moved R1 0.14 mm to (166.6, 110.5)
Routing:
- net /SCK_D13: track 35.1 -> 57.6 mm, vias 0 -> 1
- net /RESET: track 31.2 -> 12.6 mm
- net /MOSI_D11: track 45.6 -> 51.8 mm
- net /PA3_EJECT_BUTTON: track 20.0 -> 26.0 mm
- net Net-(U1-AREF): track 11.6 -> 8.27 mm
- net /MISO_D12: track 58.1 -> 55.6 mm
- net Net-(D1-K): track 4.53 -> 2.19 mm
- net /PA5_WR_PROT: track 49.9 -> 48.5 mm
- net /PD4_02: track 18.5 -> 19.8 mm
- net /PD6_RD_DATA: track 25.5 -> 24.3 mm
- net /PD7_WR_DATA: track 29.7 -> 28.6 mm
- net /PD5_03: track 11.8 -> 12.7 mm
- net Net-(J3-DAT1): track 10.8 -> 9.94 mm
- net /PD2_00: track 21.6 -> 20.9 mm
- net /PD3_01: track 19.9 -> 19.3 mm
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Other:
- board size 45.4 x 52.1 mm -> 41 x 50 mm
- board text added: "SmartPortSD SMD v1.1 github.com/djtersteegc/smartportsd-smd PCB by Chris Tersteeg Original design and code by Robert Justice, Andrea Ottaviani and Katherine Stark"
- board text added: "V1.1"
- board text removed: "SmartPortSD SMD v1.0 github.com/djtersteegc/smartportsd-smd PCB by Chris Tersteeg Original design and code by Robert Justice, Andrea Ottaviani and Katherine Stark"
- board text removed: "V1.0"
