File: smartportsd-smd.kicad_sch (KiCad schematic)
At the start: 25 parts, among them J1 DB19_Plug, J2 ICSP, J3 SD_Card_Push_Pull, SW1 SW_SPST, U1 ATmega328P-A, U2 4050, U3 AMS1117-3.3, Y1 16MHz

Commit message: Version 1.1
Parts:
- J1: footprint Tersteeg:DSUB-19_Male_Vertical_P2.77x2.84mm_MountingHoles -> Tersteeg:DSUB-19_Male_Vertical_P2.77x2.84mm_Narrow_MountingHoles
Changed lines of the file:
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@@
   (title_block
     (title "SmartPortSD SMD")
-    (date "2023-12-04")
-    (rev "v1.0")
+    (date "2023-12-07")
+    (rev "v1.1")
     (company "Chris Tersteeg")
   )
@@
       (effects (font (size 1.27 1.27)))
     )
-    (property "Footprint" "Tersteeg:DSUB-19_Male_Vertical_P2.77x2.84mm_MountingHoles" (at 41.91 138.43 0)
-      (effects (font (size 1.27 1.27)) hide)
-    )
+    (property "Footprint" "Tersteeg:DSUB-19_Male_Vertical_P2.77x2.84mm_Narrow_MountingHoles" (at 41.91 138.43 0)
+      (effects (font (size 1.27 1.27)) hide)
+    )
